File: coroam_brains/coroam_brains.kicad_pcb (KiCad board)
At the start: 2 copper layers, 19 parts, among them U1 L7805, U2 mini_esp32

Commit message: finishing brains schematics
Parts:
- added C6: 22u, Capacitor_THT:CP_Radial_D5.0mm_P2.50mm, F.Cu at (58.5, 85.5)
- added C7: 22u, Capacitor_THT:CP_Radial_D5.0mm_P2.50mm, F.Cu at (46.5, 85.5)
- added C8: 22u, Capacitor_THT:CP_Radial_D5.0mm_P2.50mm, F.Cu at (70.5, 86.0)
- added CaseFan1: Fan_4pin, Connector:FanPinHeader_1x04_P2.54mm_Vertical, F.Cu at (68.0, 93.0)
- added D3: D_Small_ALT, Diode_SMD:D_SMB_Handsoldering, F.Cu at (71.0, 99.5)
- added D4: D_Small_ALT, Diode_SMD:D_SMB_Handsoldering, F.Cu at (47.0, 99.5)
- added D5: D_Small_ALT, Diode_SMD:D_SMB_Handsoldering, F.Cu at (59.0, 99.5)
- added J1: OpenCirc, Connector_PinSocket_2.54mm:PinSocket_1x03_P2.54mm_Vertical, F.Cu at (132.0, 99.5)
- added J2: 12V_in, TerminalBlock_Phoenix:TerminalBlock_Phoenix_PT-1,5-2-5.0-H_1x02_P5.00mm_Horizontal, F.Cu at (47.5, 113.0)
- added Pump1: Fan_4pin, Connector:FanPinHeader_1x04_P2.54mm_Vertical, F.Cu at (56.0, 93.0)
- added R10: 5.1k, Resistor_SMD:R_2010_5025Metric_Pad1.52x2.65mm_HandSolder, F.Cu at (73.5, 105.5)
- added R11: 5.1k, Resistor_SMD:R_2010_5025Metric_Pad1.52x2.65mm_HandSolder, F.Cu at (61.5, 105.5)
- added R12: 10k, Resistor_SMD:R_2010_5025Metric_Pad1.52x2.65mm_HandSolder, F.Cu at (44.5, 105.5)
- added R13: 10k, Resistor_SMD:R_2010_5025Metric_Pad1.52x2.65mm_HandSolder, F.Cu at (68.5, 105.5)
- added R14: 10k, Resistor_SMD:R_2010_5025Metric_Pad1.52x2.65mm_HandSolder, F.Cu at (56.5, 105.5)
- added R3: 10k, Resistor_SMD:R_2010_5025Metric_Pad1.52x2.65mm_HandSolder, F.Cu at (136.7, 101.0)
- added R4: 5.1k, Resistor_SMD:R_2010_5025Metric_Pad1.52x2.65mm_HandSolder, F.Cu at (142.5, 103.5)
- added R5: 10k, Resistor_SMD:R_2010_5025Metric_Pad1.52x2.65mm_HandSolder, F.Cu at (142.5, 99.0)
- added R6: 10k, Resistor_SMD:R_2010_5025Metric_Pad1.52x2.65mm_HandSolder, F.Cu at (50.5, 85.5)
- added R7: 10k, Resistor_SMD:R_2010_5025Metric_Pad1.52x2.65mm_HandSolder, F.Cu at (74.5, 85.5)
- added R8: 10k, Resistor_SMD:R_2010_5025Metric_Pad1.52x2.65mm_HandSolder, F.Cu at (62.5, 85.5)
- added R9: 5.1k, Resistor_SMD:R_2010_5025Metric_Pad1.52x2.65mm_HandSolder, F.Cu at (49.5, 105.5)
- added RadiatorFan1: Fan_4pin, Connector:FanPinHeader_1x04_P2.54mm_Vertical, F.Cu at (44.0, 93.0)
- C1, C2, C3: value 4.7u -> 22u
- C4: footprint Capacitor_THT:CP_Radial_D5.0mm_P2.50mm -> Capacitor_SMD:C_1206_3216Metric_Pad1.42x1.75mm_HandSolder
- C5: footprint Capacitor_THT:CP_Radial_D5.0mm_P2.50mm -> Capacitor_SMD:C_0603_1608Metric_Pad1.05x0.95mm_HandSolder
- D1: value Red -> 5V
- D2: value Green -> 12V
- R1, R2: footprint Resistor_THT:R_Axial_DIN0414_L11.9mm_D4.5mm_P15.24mm_Horizontal -> Resistor_THT:R_Axial_DIN0207_L6.3mm_D2.5mm_P7.62mm_Horizontal
- moved D1 112.6 mm to (44.5, 123.0), turned to 270 degrees
- moved lls1 104.7 mm to (70.5, 117.0), turned to 180 degrees
- moved C1 98.5 mm to (74.0, 136.0), turned to 90 degrees
- moved D2 93.0 mm to (56.0, 117.5), turned to 270 degrees
- moved C2 91.0 mm to (74.0, 127.0), turned to 270 degrees
- moved C5 87.3 mm to (62.0, 133.5), turned to 180 degrees
- moved C3 84.3 mm to (55.0, 111.0), turned to 270 degrees
- moved R1 82.6 mm to (46.0, 128.5), turned to 270 degrees
- moved C4 81.5 mm to (57.5, 133.5)
- moved U1 68.0 mm to (57.0, 127.5), turned to 90 degrees
- moved LCD_I2C1 66.8 mm to (112.5, 95.0)
- moved R2 63.9 mm to (61.5, 119.0), turned to 90 degrees
- moved TempCasing1 45.7 mm to (168.5, 122.0)
- moved TempLaser1 39.4 mm to (168.5, 130.5)
- moved TempWater1 39.1 mm to (168.5, 113.5)
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Connections:
- U2 pad 10: Net-(U2-Pad10) -> RadFanPWM_3V
- U2 pad 26: Net-(U2-Pad26) -> Door_3V
- U2 pad 5: Net-(U2-Pad5) -> PumpTach_3V
- U2 pad 6: Net-(U2-Pad6) -> PumpPWM_3V
- U2 pad 7: Net-(U2-Pad7) -> CaseFanTach_3V
- U2 pad 8: Net-(U2-Pad8) -> CaseFanPWM_3V
- U2 pad 9: Net-(U2-Pad9) -> RadFanTach_3V
- lls1 pad 11: Net-(lls1-Pad11) -> PumpPWM
- lls1 pad 2: Net-(lls1-Pad2) -> PumpPWM_3V
- lls1 pad 5: Net-(lls1-Pad5) -> CaseFanPWM_3V
- lls1 pad 6: Net-(lls1-Pad6) -> RadFanPWM_3V
- lls1 pad 7: Net-(lls1-Pad7) -> RadFanPWM
- lls1 pad 8: Net-(lls1-Pad8) -> CaseFanPWM
Routing:
- net +12V: track 0.00 -> 29.9 mm
- net RadFanTach: track 0.00 -> 20.8 mm, vias 0 -> 1
- net PumpTach: track 0.00 -> 20.8 mm, vias 0 -> 1
- net CaseFanTach: track 0.00 -> 20.8 mm, vias 0 -> 1
- net Door_5V: track 0.00 -> 8.77 mm
- net RadFanTach_3V: track 0.00 -> 5.00 mm
- net PumpTach_3V: track 0.00 -> 5.00 mm
- net CaseFanTach_3V: track 0.00 -> 5.00 mm
- net Door_3V: track 0.00 -> 4.50 mm
Other:
- rule pad_to_mask_clearance: 0.051 -> 0
- rule solder_mask_min_width: 0.25 -> 0.1
- rule trace_min: 0.2 -> 0.1
- rule via_min_drill: 0.3 -> 0.2
- rule via_min_size: 0.4 -> 0.45
- board text added: "Door"
- board text added: "In"
- board text added: "Out"
